File: board/BattGuard/BattGuard.kicad_sch (KiCad schematic)
At the start: 0 parts

Commit message: 10.15.2026
Parts:
- added C1: 1 uF, symbol Device:C
- added C2: 100 uF, symbol Device:C_US
- added J1: OQ0271510000G, OQ0271510000G:AMPHENOL_OQ0271510000G, symbol BattGuard:OQ0271510000G
- added R1: 2.4, symbol Device:R_US
- added U1: BQ25756ERRVR, BQ25756ERRVR:IC_BQ25756ERRVR, symbol BattGuard:BQ25756ERRVR
- added U2: ESP32-S3-WROOM-1, RF_Module:ESP32-S3-WROOM-1, symbol RF_Module:ESP32-S3-WROOM-1
- added U3: LM317_TO3, Package_TO_SOT_THT:TO-3, symbol Regulator_Linear:LM317_TO3
Connections:
- new net: C2.1, R1.2
- new net: U2.1 (GND), U2.40 (GND), U2.41 (GND)
- new net: U1.15 (NC), U1.16 (NC), U1.31 (NC)
- new net GND: C1.2, C2.2
- new net PGND: U1.17 (PGND), U1.22 (PGND), U1.37 (PGND)
- new net VAC: C1.1, J1.2, R1.1, U1.32 (VAC), U1.33 (VAC)
Other:
- note added: "GND"
- note added: "VIN"

Commit message: 10.16.2026
Parts:
- added C10, C11, C9: 10uF, symbol Device:C
- added C12: 1uF, symbol Device:C
- added C13: 100nF, symbol Device:C
- added C14: 100pF, symbol Device:C
- added C15: 470nF, symbol Device:C
- added C16, C17: 100nF 100V, symbol Device:C
- added C18, C19, C8: 4.7uF, symbol Device:C
- added C3: 4.7, symbol Device:C_US
- added C4, C5, C6: 56uF, symbol Device:C_US
- added C7: 4.7 uF, symbol Device:C
- added R2: 5m, symbol Device:R_US
- added R3, R4, R8: 10, symbol Device:R_US
- added R5: 1 M, symbol Device:R_US
- added R6: 73.2k, symbol Device:R_US
- added R7: 27.4k, symbol Device:R_US
Connections:
- net PGND is gone; now on net GND: U1.17 (PGND), U1.22 (PGND), U1.37 (PGND)
- net GND: now also J1.1, C10.2, C11.2, C12.2, C13.2, C14.2, C16.2, C17.1, C18.2, C19.2, C3.2, C4.2, C5.2, C6.2, C7.2, C8.2, C9.2, R7.2
- net VAC: now also C3.1, C4.1, C5.1, R2.1, R3.1, R5.1
- net at U1.23 (DRV_SUP): now also C19.1, R8.2
- net at U1.24 (REGN): now also C18.1, R8.1
- net at U1.29 (ACN): now also C15.2, C16.1, R4.2
- net at U1.30 (ACP): now also C15.1, C17.2, R3.2
- net at U1.34 (ACUV): now also R5.2, R6.1
- net at U1.35 (ACOV): now also R6.2, R7.1
- new net Vsys: C10.1, C11.1, C12.1, C13.1, C14.1, C6.1, C7.1, C8.1, C9.1, R2.2, R4.1
- no-connect marks 0 -> 1
Other:
- moved on the sheet: C1, C2, J1, R1, U1, U2, U3

Commit message: 10.17.2026
Parts:
- removed U2: ESP32-S3-WROOM-1, RF_Module:ESP32-S3-WROOM-1, symbol RF_Module:ESP32-S3-WROOM-1
- removed U3: LM317_TO3, Package_TO_SOT_THT:TO-3, symbol Regulator_Linear:LM317_TO3
- added BT1: 4s 6500mah 130c 16.8v-14v, symbol Device:Battery
- added C20: 4.7 uF, symbol Device:C
- added C21: 4.7uF, symbol Device:C
- added C22, C23, C24: 10uF, symbol Device:C
- added C25: 1uF, symbol Device:C
- added C26, C29, C30, C39: 100nF, symbol Device:C
- added C27: 100pF, symbol Device:C
- added C28: 56uF, 80V, symbol Device:C_US
- added C31: 470nF, symbol Device:C
- added C32, C33: 100, symbol Device:C
- added C34, C35: 56uF 80V, symbol Device:C_US
- added C36: 1uF 100v, symbol Device:C
- added C37: 100nF 100v, symbol Device:C
- added C38: 1nF 100v, symbol Device:C
- added C40: 220uF 35v, symbol Device:C_US
- added C41, C42: .1 uF, symbol Device:C
- added D1, D2: B560C-13-F, B560C-13-F:SMC, symbol BattGuard:B560C-13-F
- added D3, D4: V1FM10-M3_H, V1FM10-M3_H:DIO_V1FM10-M3_H, symbol BattGuard:V1FM10-M3_H
- added J2: Barrel_Jack, symbol Connector:Barrel_Jack
- added J3, J4: Conn_01x22_Pin, symbol Connector:Conn_01x22_Pin
- added J5: Conn_01x02_Pin(xt60), symbol Connector:Conn_01x02_Pin
- added J6: OLED DISPLAY, symbol Connector:Conn_01x05_Pin
- added L1: IHLP6767GZER6R8M01 10uH, IHLP6767GZER6R8M01:IND_IHLP6767GZER6R8M01, symbol BattGuard:IHLP6767GZER6R8M01
- added Q1, Q2, Q3, Q4: SIR680LDP-T1-RE3, SIR680LDP-T1-RE3:TRANS_SIR680LDP-T1-RE3, symbol BattGuard:SIR680LDP-T1-RE3
- added Q5, Q6: PMOS, symbol Simulation_SPICE:PMOS
- added Q7: NMOS, symbol Simulation_SPICE:NMOS
- added R10, R9: 10, symbol Device:R_US
- added R11: 5m, symbol Device:R_US
- added R12: 133k, symbol Device:R_US
- added R13: 249k, symbol Device:R_US
- added R14: 25.8k, symbol Device:R_US
- added R15: 5.24k, symbol Device:R_US
- added R16: 30.1k, symbol Device:R_US
- added R17, R23: 4.7k, symbol Device:R_US
- added R18: 240, symbol Device:R_US
- added R19: 100, symbol Device:R_US
- added R20, R21: 100k, symbol Device:R_US
- added R22: .1, symbol Device:R_US
- added R24, R25, R26, R27, R28, R29: 10k, symbol Device:R_US
- added TH1(103AT-2): 10k, symbol Device:Thermistor_NTC
- added U3: MCP45HV51-ST, Package_SO:TSSOP-14_4.4x5mm_P0.65mm, symbol Potentiometer_Digital:MCP45HV51-ST
- added U4: INA226, Package_SO:TSSOP-10_3x3mm_P0.5mm, symbol Sensor_Energy:INA226
- added U5: LM317_TO3, Package_TO_SOT_THT:TO-3, symbol Regulator_Linear:LM317_TO3
- C6: value 56uF -> 56uF, 80V
- R6: value 73.2k -> 249k
- R7: value 27.4k -> 32.4k
Connections:
- net GND: now also C1.1, U1.10 (ILIM_HIZ), U1.9 (ICHG), BT1.2 (-), C20.2, C21.2, C22.2, C23.2, C24.2, C25.2, C26.2, C27.2, C28.2, C32.1, C33.2, C34.2, C35.2, C36.2, C37.2, C38.2, C39.2, C40.2, C41.2, C42.2, J2.2, J5.2 (Pin_2), J6.1 (Pin_1), Q2.1, Q2.2, Q2.3, Q3.1, Q3.2, Q3.3, Q7.3 (S), R12.1, R16.2, R20.2, TH1(103AT-2).2, U3.10 (V-), U3.11 (P0B), U3.3 (A1), U3.5 (A0), U3.6 (~{WLAT}), U3.9 (DGND), U4.1 (A1), U4.2 (A0), U4.7 (GND); no longer C1.2
- net VAC: now also C1.2, D1.C, D2.C; no longer C1.1, J1.2
- net Vsys: now also Q1.D
- net REGN: now reaches C18.1, R8.1, U1.24 (REGN)
- net REGN: now also R15.1
- net at C19.1, R8.2, U1.23 (DRV_SUP): now also D3.2, D4.2
- net GPIO9: now reaches U1.1 (SCL)
- net GPIO9: now also J3.15 (Pin_15), R23.2, U3.2 (SCL)
- net FBG: now reaches U1.11 (FBG)
- net FBG: now also R14.1
- net at U1.12 (FB): now also R13.1, R14.2
- net at U1.13 (SRN): now also C31.1, C33.1, R10.2
- net at U1.14 (SRP): now also C31.2, C32.2, R9.2
- net at U1.18 (SW2): now also L1.2, Q4.3
- net HIDRV2: now reaches U1.19 (HIDRV2)
- net HIDRV2: now also Q4.4
- net GPIO8: now reaches U1.2 (SDA)
- net GPIO8: now also J3.12 (Pin_12), R17.2, U3.4 (SDA)
- net BTST2: now reaches U1.20 (BTST2)
- net BTST2: now also C30.2, D4.1
- net LODRV2: now reaches U1.21 (LODRV2)
- net LODRV2: now also Q3.4
- net LODRV1: now reaches U1.25 (LODRV1)
- net LODRV1: now also Q2.4
- net at U1.26 (BTST1): now also C29.1, D3.1
- net HIDRV1: now reaches U1.27 (HIDRV1)
- net HIDRV1: now also Q1.4
- net at U1.28 (SW1): now also Q1.2
- net GPIO11: now reaches U1.3 (~{INT})
- net GPIO11: now also U1.4 (STAT1), U1.5 (STAT2), J3.17 (Pin_17), J3.18 (Pin_18), J3.19 (Pin_19), J3.20 (Pin_20), R25.2, R26.2, R27.2, R28.2, U4.3 (~{Alert})
- net at U1.36 (FSW_SYNC): now also R12.2
- net GPIO10: now reaches U1.7 (~{CE})
- net GPIO10: now also J3.16 (Pin_16), R24.2
- net TS: now reaches U1.8 (TS)
- net TS: now also R15.2, R16.1, TH1(103AT-2).1
- new net: Q5.3 (S), Q6.3 (S), R21.1
- new net: Q5.2 (G), Q6.2 (G), Q7.1 (D), R21.2
- new net: C29.2, Q1.3
- new net: L1.1, Q1.1, Q2.D
- new net: Q7.2 (G), R19.2, R20.1
- new net: J4.21 (Pin_21), J4.22 (Pin_22)
- new net: D2.A, J2.1
- new net: Q3.D, Q4.2
- new net: D1.A, J1.2
- new net: C30.1, Q4.1
- new net: C42.1, Q6.1 (D), R22.1, U4.10 (Vin+)
- new net: U3.12 (P0W), U5.1 (ADJ)
- new net: Q5.1 (D), R18.1, U5.3 (VO)
- new net: R18.2, U3.13 (P0A)
- new net: J5.1 (Pin_1), R22.2, U4.8 (Vbus), U4.9 (Vin-)
- new net 3v3: J3.1 (Pin_1), J3.2 (Pin_2), J6.2 (Pin_2), R17.1, R23.1, R24.1, R25.1, R26.1, R27.1, R28.1, R29.1
- new net Chip_PU: J3.3 (Pin_3)
- new net GNDREF: J4.1 (Pin_1)
- new net GPI15: J3.8 (Pin_8)
- new net GPI16: J3.9 (Pin_9)
- new net GPIO0: J4.14 (Pin_14)
- new net GPIO1: J4.4 (Pin_4)
- new net GPIO17: J3.10 (Pin_10)
- new net GPIO18: J3.11 (Pin_11)
- new net GPIO19: J4.20 (Pin_20)
- new net GPIO2: J4.5 (Pin_5)
- new net GPIO20: J4.19 (Pin_19)
- new net GPIO21: J4.18 (Pin_18)
- new net GPIO3: J3.13 (Pin_13)
- new net GPIO35: J4.13 (Pin_13)
- new net GPIO36: J4.12 (Pin_12)
- new net GPIO37: J4.11 (Pin_11)
- new net GPIO38: J4.10 (Pin_10)
- new net GPIO39: J4.9 (Pin_9)
- new net GPIO4: J3.4 (Pin_4), R19.1
- new net GPIO40: J4.8 (Pin_8)
- new net GPIO41: J4.7 (Pin_7)
- new net GPIO42: J4.6 (Pin_6)
- new net GPIO45: J4.15 (Pin_15)
- new net GPIO46: J3.14 (Pin_14)
- new net GPIO47: J4.17 (Pin_17)
- new net GPIO48: J4.16 (Pin_16)
- new net GPIO5: J3.5 (Pin_5), J6.3 (Pin_3)
- new net GPIO6: J3.6 (Pin_6), J6.4 (Pin_4)
- new net GPIO7: J3.7 (Pin_7), J6.5 (Pin_5), R29.2
- new net Pout: C20.1, C21.1, C22.1, C23.1, C24.1, C25.1, C26.1, C27.1, C28.1, Q4.D, R11.1, R9.1
- new net U0RXD: J4.3 (Pin_3)
- new net U0TXD: J4.2 (Pin_2)
- new net VCC_5V: J3.21 (Pin_21)
- new net Vsystem: BT1.1 (+), C34.1, C35.1, C36.1, C37.1, C38.1, C39.1, C40.1, C41.1, R10.1, R11.2, R13.2, U3.14 (V+), U5.2 (VI)
- no-connect marks 1 -> 2
Other:
- note added: "+"
- note added: "-"
- note added: "3v3"
- note added: "Trickle Charge Port"
- note added: "esp enable gpio 1=charging, 0= no charge"
- note added: "i2c"
- note added: "shunt"
- moved on the sheet: C10, C11, C12, C13, C14, C15, C16, C17, C18, C19, C2, C3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

Commit message: 10.17.2026 night
Connections:
- net GND: now also J3.22 (Pin_22), J4.21 (Pin_21), J4.22 (Pin_22)
- net GPIO8: now also U4.4 (SDA)
- net GPIO9: now also U4.5 (SCL)
- net Vsystem: no longer C41.1, U3.14 (V+), U5.2 (VI)
- new net: C41.1, U3.14 (V+), U5.2 (VI)
Other:
- note added: "will be boost output"
- note removed: "i2c"
Changed lines of the file:
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@@
 		)
 	)
-	(text "i2c"
-		(exclude_from_sim no)
-		(at 193.04 227.584 0)
-		(effects
-			(font
-				(size 1.27 1.27)
-			)
-		)
-	)
 	(text "GND\n"
 		(exclude_from_sim no)
@@
 		)
 	)
-	(text "i2c"
+	(text "will be boost output\n"
 		(exclude_from_sim no)
-		(at 193.04 224.79 0)
+		(at 51.562 202.438 0)
 		(effects
 			(font
@@
 	)
 	(junction
+		(at 381 179.07)
+		(diameter 0)
+		(color 0 0 0 0)
+	)
+	(junction
 		(at 201.93 50.8)
 		(diameter 0)
@@
 	(wire
 		(pts
-			(xy 337.82 179.07) (xy 350.52 179.07)
-		)
-		(stroke
-			(width 0)
-			(type default)
-		)
-	)
-	(wire
-		(pts
 			(xy 212.09 43.18) (xy 222.25 43.18)
 		)
@@
 	(wire
 		(pts
+			(xy 331.47 179.07) (xy 350.52 179.07)
+		)
+		(stroke
+			(width 0)
+			(type default)
+		)
+	)
+	(wire
+		(pts
 			(xy 102.87 50.8) (xy 102.87 53.34)
 		)
@@
 	(wire
 		(pts
+			(xy 196.85 227.33) (xy 190.5 227.33)
+		)
+		(stroke
+			(width 0)
+			(type default)
+		)
+	)
+	(wire
+		(pts
 			(xy 335.28 64.77) (xy 345.44 64.77)
 		)
@@
 	(wire
 		(pts
+			(xy 196.85 224.79) (xy 190.5 224.79)
+		)
+		(stroke
+			(width 0)
+			(type default)
+		)
+	)
+	(wire
+		(pts
 			(xy 372.11 146.05) (xy 374.65 146.05)
 		)
@@
 		)
 	)
-	(label "Vsystem"
-		(at 45.72 204.47 0)
-		(effects
-			(font
-				(size 1.27 1.27)
-			)
-			(justify left bottom)
-		)
-	)
 	(label "GPIO13"
 		(at 337.82 171.45 0)
@@
 		)
 	)
+	(label "GPIO8"
+		(at 196.85 224.79 0)
+		(effects
+			(font
+				(size 1.27 1.27)
+			)
+			(justify left bottom)
+		)
+	)
 	(label "GPIO14"
 		(at 193.04 232.41 0)
@@
 		)
 	)
+	(label "GPIO9"
+		(at 196.85 227.33 0)
+		(effects
+			(font
+				(size 1.27 1.27)
+			)
+			(justify left bottom)
+		)
+	)
 	(label "TS"
 		(at 21.59 180.34 0)
@@
 	)
 	(symbol
+		(lib_id "power:GND")
+		(at 381 179.07 0)
+		(unit 1)
+		(body_style 1)
+		(exclude_from_sim no)
+		(in_bom yes)
+		(on_board yes)
+		(in_pos_files yes)
+		(dnp no)
+		(fields_autoplaced yes)
+		(property "Reference" "#PWR025"
+			(at 381 185.42 0)
+			(hide yes)
+			(show_name no)
+			(do_not_autoplace no)
+			(effects
+				(font
+					(size 1.27 1.27)
+				)
+			)
+		)
+		(property "Value" "GND"
+			(at 381 184.15 0)
+			(show_name no)
+			(do_not_autoplace no)
+			(effects
+				(font
+					(size 1.27 1.27)
+				)
+			)
+		)
+		(property "Footprint" ""
+			(at 381 179.07 0)
+			(hide yes)
+			(show_name no)
+			(do_not_autoplace no)
+			(effects
+				(font
+					(size 1.27 1.27)
+				)
+			)
+		)
+		(property "Datasheet" ""
+			(at 381 179.07 0)
+			(hide yes)
+			(show_name no)
+			(do_not_autoplace no)
+			(effects
+				(font
+					(size 1.27 1.27)
+				)
+			)
+		)
+		(property "Description" "Power symbol creates a global label with name \"GND\" , ground"
+			(at 381 179.07 0)
+			(hide yes)
+			(show_name no)
+			(do_not_autoplace no)
+			(effects
+				(font
+					(size 1.27 1.27)
+				)
+			)
+		)
+		(pin "1"
+		)
+		(instances
+			(project "BattGuard"
+				(path "/236cbdd7-d83d-4a8e-9ca8-a6b8cdb61d8b"
+					(reference "#PWR025")
+					(unit 1)
+				)
+			)
+		)
+	)
+	(symbol
 		(lib_id "Connector:Conn_01x22_Pin")
 		(at 367.03 151.13 0)
@@
 					(unit 1)
 				)
+			)
+		)
+	)
+	(symbol
+		(lib_id "power:GND")
+		(at 331.47 179.07 0)
+		(unit 1)
+		(body_style 1)
+		(exclude_from_sim no)
+		(in_bom yes)
+		(on_board yes)
+		(in_pos_files yes)
+		(dnp no)
+		(fields_autoplaced yes)
+		(property "Reference" "#PWR023"
+			(at 331.47 185.42 0)
+			(hide yes)
+			(show_name no)
+			(do_not_autoplace no)
+			(effects
+				(font
+					(size 1.27 1.27)
+				)
+			)
+		)
+		(property "Value" "GND"
+			(at 331.47 184.15 0)
+			(show_name no)
+			(do_not_autoplace no)
+			(effects
+				(font
+					(size 1.27 1.27)
+				)
+			)
+		)
+		(property "Footprint" ""
+			(at 331.47 179.07 0)
+			(hide yes)
+			(show_name no)
+			(do_not_autoplace no)
+			(effects
+				(font
+					(size 1.27 1.27)
+				)
+			)
+		)
+		(property "Datasheet" ""
+			(at 331.47 179.07 0)
+			(hide yes)
+			(show_name no)
+			(do_not_autoplace no)
+			(effects
+				(font
+					(size 1.27 1.27)
+				)
+			)
+		)
+		(property "Description" "Power symbol creates a global label with name \"GND\" , ground"
+			(at 331.47 179.07 0)
+			(hide yes)
+			(show_name no)
+			(do_not_autoplace no)
+			(effects
+				(font
+					(size 1.27 1.27)
+				)
+			)
+		)
+		(pin "1"
+		)
+		(instances
+			(project "BattGuard"
+				(path "/236cbdd7-d83d-4a8e-9ca8-a6b8cdb61d8b"
+					(reference "#PWR023")
+					(unit 1)
+				)

Commit message: 10.18.2026 Schematic v1
Parts:
- removed Q5, Q6: PMOS, symbol Simulation_SPICE:PMOS
- removed Q7: NMOS, symbol Simulation_SPICE:NMOS
- added C43, C56: 100nF, symbol Device:C
- added C44, C45: 22uF 16V, symbol Device:C_US
- added C46, C47: 4.7uF 50V, symbol Device:C_US
- added C48: 100nF 50V, symbol Device:C_US
- added C49: 1uF 16V, symbol Device:C_US
- added C50: 2.2 uF 10V, symbol Device:C
- added C51, C53, C54: 10uF 50V, symbol Device:C
- added C52: 1uF 50V, symbol Device:C
- added C57: 10uF 16V, symbol Device:C
- added D10, D11, D7, D8, D9: LED, symbol Device:LED
- added D5: B560C-13-F, B560C-13-F:SMC, symbol BattGuard:B560C-13-F
- added D6: Blue LED, symbol Device:LED
- added F1: MF-MSMF150-2, MF-MSMF150-2:FUSER_MF-MSMF150-2, symbol BattGuard:MF-MSMF150-2
- added J10, J11, J12, J13, J14, J9: Conn_01x01_Pin, symbol Connector:Conn_01x01_Pin
- added J7: EC5 JUMP CONNECTOR, symbol Connector:Conn_01x02_Pin
- added J8: GSB4111312HR, GSB4111312HR:AMPHENOL_GSB4111312HR, symbol BattGuard:GSB4111312HR
- added L3, L4: SRP5030TA-100M, IND_SRP5030TA_BRN, symbol BattGuard:SRP5030TA-100M
- added Q7, Q9: AO3401A, Package_TO_SOT_SMD:SOT-23, symbol Transistor_FET:AO3401A
- added Q8: 2N7002, Package_TO_SOT_SMD:SOT-23, symbol Transistor_FET:2N7002
- added R30: 100k, symbol Device:R_US
- added R31: 13.7k, symbol Device:R_US
- added R32: 845k, symbol Device:R_US
- added R33: 60.4k, symbol Device:R_US
- added R34, R35, R36, R37, R38, R39, R40, R41, R45, R46, R47, R48, R49: 1k, symbol Device:R_US
- added R42, R43: 10k, symbol Device:R_US
- added R44: 100, symbol Device:R_US
- added SW1, SW2: SW_Push, symbol Switch:SW_Push
- added U2: LMR51420XDDCR, SOT23_DDC_TEX, symbol BattGuard:LMR51420XDDCR
- added U6: TLV76133KVUR, Package_TO_SOT_SMD:SOT-223-3_TabPin2, symbol Regulator_Linear:TLV76133DCY
- added U7: TLV61047DDC, Package_TO_SOT_SMD:SOT-23-5, symbol Regulator_Switching:TLV61047DDC
Connections:
- net GNDREF is gone; now on net -BATT: J4.1 (Pin_1)
- net 3v3: no longer J3.1 (Pin_1), J3.2 (Pin_2), R17.1, R23.1, R24.1, R25.1, R26.1, R27.1, R28.1, R29.1
- net GPIO1: now also R34.1
- net GPIO17: now also R48.1
- net GPIO18: now also R49.1
- net GPIO2: now also R35.1
- net GPIO21: now also R44.1
- net GPIO39: now also R45.1
- net GPIO40: now also R42.2, SW1.1
- net GPIO41: now also R39.1
- net GPIO42: now also R38.1
- net GPIO47: now also R43.2, SW2.1
- net Vsystem: now also C46.1, C47.1, C48.1, C51.1, J7.1 (Pin_1), L3.2, U2.3 (VIN), U2.5 (EN), U7.4 (EN), U7.5 (VIN)
- net at R21.1: now also Q7.2 (S), Q9.2 (S)
- net at R21.2: now also Q7.1 (G), Q8.3 (D), Q9.1 (G)
- net +18.5V: now reaches C41.1, U3.14 (V+), U5.2 (VI)
- net +18.5V: now also C52.1, C53.1, C54.1, D5.C
- net at R19.2, R20.1: now also Q8.1 (G)
- net at C42.1, R22.1, U4.10 (Vin+): now also Q9.3 (D)
- net at R18.1, U5.3 (VO): now also Q7.3 (D)
- net +3.3V: now reaches U4.6 (VS)
- net +3.3V: now also R17.1, R23.1, R24.1, R25.1, R26.1, R27.1, R28.1, R29.1, U3.1 (VL), U3.8 (~{SHDN})
- net +BATT: now reaches J5.1 (Pin_1), R22.2, U4.8 (Vbus), U4.9 (Vin-)
- net GND renamed -BATT
- net -BATT: now also C44.2, C45.2, C46.2, C47.2, C48.2, C49.2, C50.2, C51.2, C52.2, C53.2, C54.2, C56.2, C57.2, D10.1 (K), D11.1 (K), D6.1 (K), D7.1 (K), D8.1 (K), D9.1 (K), J7.2 (Pin_2), J8.4 (GND), J8.7 (GND_DRAIN), J8.SH1 (SHIELD), J8.SH2 (SHIELD__1), Q8.2 (S), R31.1, R33.2, SW1.2, SW2.2, U2.1 (GND), U6.1 (GND), U7.2 (GND)
- net Pout renamed Vout
- net VCC_5V renamed +5V
- net +5V: now also C44.1, C45.1, C49.1, F1.1, J14.1 (Pin_1), L4.1, R30.2, U6.3 (VI)
- new net: D5.A, L3.1, R32.1, U7.1 (SW)
- new net: J11.1 (Pin_1), R38.2, R40.1
- new net: R32.2, R33.1, U7.3 (FB)
- new net: C56.1, C57.1, F1.2, J8.1 (VBUS)
- new net: D11.2 (A), R49.2
- new net: D7.2 (A), R45.2
- new net: C43.1, L4.2, U2.2 (SW)
- new net: D10.2 (A), R48.2
- new net: D6.2 (A), R44.2
- new net: J12.1 (Pin_1), R39.2, R41.2
- new net: D8.2 (A), R46.2
- new net: J10.1 (Pin_1), R35.2, R37.2
- new net: J8.2 (D-), J8.3 (D+)
- new net: R30.1, R31.2, U2.4 (FB)
- new net: J9.1 (Pin_1), R34.2, R36.1
- new net: D9.2 (A), R47.2
- new net: J3.1 (Pin_1), J3.2 (Pin_2)
- new net: C43.2, U2.6 (CB)
- new net +3V3: C50.1, J13.1 (Pin_1), R36.2, R37.1, R40.2, R41.1, R42.1, R43.1, U6.2 (VO)
- new net GPIO15: R46.1
- new net GPIO16: R47.1
- no-connect marks 2 -> 6
Other:
- note added: "12V CHARGE CIRCUIT"
- note added: "3v3 LDO"
- note added: "5V BUCK LMR51420"
- note added: "Boost Circuit TLV76133KVUR"
- note added: "ESP32-S3-DEVKITC-1 HEADER"
- note added: "USB CIRCUIT"
- note removed: "3v3"
- note removed: "shunt"
- note removed: "will be boost output"
- moved on the sheet: BT1, C1, C10, C11, C12, C13, C14, C15, C16, C17, C18, C19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

Commit message: 10.18.2026 update
Parts:
- BT1, J2, J5, J6, J7, SW1, SW2: now left out of the parts list
- C1, C10, C11, C12, C13, C14, C15, C16, C17, C18, C19, C2, C20, C21, C22, C23, C24, C25, C26, C27, C29, C3, C30, C31, C36, C37, C38, C39, C41, C42, C43, C46, C47, C48, C49, C50, C51, C52, C53, C54, C56, C57, C7, C8, C9: footprint (none) -> Capacitor_SMD:C_0805_2012Metric
- C28, C34, C35, C4, C40, C44, C45, C5, C6: footprint (none) -> Capacitor_THT:CP_Radial_D10.0mm_P2.50mm
- C32, C33: value 100 -> 100nF; footprint (none) -> Capacitor_SMD:C_0805_2012Metric
- D1, D2, D5: footprint B560C-13-F:SMC -> Diode_SMD:D_SMC
- D10, D11, D6, D7, D8, D9, J10, J11, J12, J13, J14, J9: footprint (none) -> TestPoint:TestPoint_Pad_1.0x1.0mm
- D3, D4: footprint V1FM10-M3_H:DIO_V1FM10-M3_H -> Diode_SMD:D_SMC
- F1: footprint MF-MSMF150-2:FUSER_MF-MSMF150-2 -> Fuse:Fuse_1812_4532Metric
- J1: footprint OQ0271510000G:AMPHENOL_OQ0271510000G -> BattGuard:AMPHENOL_OQ0271510000G
- J3, J4: footprint (none) -> Connector_PinHeader_2.00mm:PinHeader_1x22_P2.00mm_Vertical
- J8: footprint GSB4111312HR:AMPHENOL_GSB4111312HR -> Connector_USB:USB3_A_Receptacle_Wuerth_692122030100
- L1: footprint IHLP6767GZER6R8M01:IND_IHLP6767GZER6R8M01 -> Inductor_SMD:L_Vishay_IHLP-6767
- L3, L4: footprint IND_SRP5030TA_BRN -> Inductor_SMD:L_Bourns_SRP5030T
- Q1, Q2, Q3, Q4: footprint SIR680LDP-T1-RE3:TRANS_SIR680LDP-T1-RE3 -> BattGuard:TRANS_SIR680LDP-T1-RE3
- R1, R10, R11, R12, R13, R14, R15, R16, R17, R18, R19, R2, R20, R21, R22, R23, R24, R25, R26, R27, R28, R29, R3, R30, R31, R32, R33, R34, R35, R36, R37, R38, R39, R4, R40, R41, R42, R43, R44, R45, R46, R47, R48, R49, R5, R6, R7, R8, R9: footprint (none) -> Resistor_SMD:R_0805_2012Metric
- TH1(103AT-2)1: renamed from TH1(103AT-2); footprint (none) -> Resistor_SMD:R_0805_2012Metric
- U1: footprint BQ25756ERRVR:IC_BQ25756ERRVR -> BattGuard:IC_BQ25756ERRVR

Commit message: 10.19.2026 pcb layout
Parts:
- added C58: 100nF, Capacitor_SMD:C_0805_2012Metric, symbol Device:C
- added C59: 10uF, Capacitor_SMD:C_0805_2012Metric, symbol Device:C
- added R50: 0, Resistor_SMD:R_0805_2012Metric, symbol Device:R_US
- J3, J4: footprint Connector_PinHeader_2.00mm:PinHeader_1x22_P2.00mm_Vertical -> Connector_PinSocket_2.54mm:PinSocket_1x22_P2.54mm_Vertical
- renumbered TH1(103AT-2)1 to TH1
Connections:
- net +3.3V is gone; now on net +3V3: R17.1, R23.1, R24.1, R25.1, R26.1, R27.1, R28.1, R29.1, U3.1 (VL), U3.8 (~{SHDN}), U4.6 (VS)
- net GPI15 is gone; now on net GPIO15: J3.8 (Pin_8)
- net GPI16 is gone; now on net GPIO16: J3.9 (Pin_9)
- net +18.5V: now also R32.1
- net +5V: now also C58.1, C59.1
- net -BATT: now also C58.2, C59.2, R50.2; no longer R12.1, R16.2, R7.2, TH1.2, U1.10 (ILIM_HIZ), U1.9 (ICHG)
- net SW1: now reaches C29.2, Q1.3
- net SW1: now also L1.1, Q1.1, Q1.2, Q2.D, U1.28 (SW1)
- net at D5.A, L3.1, U7.1 (SW): no longer R32.1
- net SW2: now reaches L1.2, Q4.3, U1.18 (SW2)
- net SW2: now also C30.1, Q3.D, Q4.1, Q4.2
- new net AGND: R12.1, R16.2, R50.1, R7.2, TH1.2, U1.10 (ILIM_HIZ), U1.9 (ICHG)
Other:
- moved on the sheet: C52, C53, C54, R33

Commit message: 10.19.2026 pcb v1 no route
Parts:
- added J15: Conn_01x01_Pin, MountingHole:MountingHole_2.2mm_M2_DIN965_Pad, symbol Connector:Conn_01x01_Pin
- added J17: S5B-XH-A, TeamLib:JST_S5B-XH-A, symbol Battguard:S5B-XH-A
- J1: footprint BattGuard:AMPHENOL_OQ0271510000G -> BattGuard:CONN_SD-39522-003_02P_MOL
- J2: footprint (none) -> Connector_BarrelJack:BarrelJack_CUI_PJ-063AH_Horizontal_CircularHoles; now in the parts list
- J5: footprint (none) -> Connector_AMASS:AMASS_XT60IPW-M_1x03_P7.20mm_Horizontal; now in the parts list
- J7: footprint (none) -> Connector_AMASS:AMASS_XT60PW-M_1x02_P7.20mm_Horizontal; now in the parts list
Connections:
- net +18.5V: now also D5.1; no longer D5.C
- net -BATT: now also J17.1
- net VAC: now also D1.1, D2.1; no longer D1.C, D2.C
- net Vsystem: now also J15.1 (Pin_1), J17.5
- net at L3.1, U7.1 (SW): now also D5.2; no longer D5.A
- net at J2.1: now also D2.2; no longer D2.A
- net at J1.2: now also D1.2; no longer D1.A
Other:
- note added: "BMS Charge + NODE"
