File: board/BattGuard/BattGuard.kicad_sch (KiCad schematic)
At the start: 159 parts, among them J1 OQ0271510000G, J10 Conn_01x01_Pin, J11 Conn_01x01_Pin, J12 Conn_01x01_Pin, J13 Conn_01x01_Pin, J15 Conn_01x01_Pin, J17 S5B-XH-A, J18 FAN1 5V, J19 FAN2 5V, J2 Barrel_Jack, J3 Conn_01x22_Pin, J4 Conn_01x22_Pin, J5 Conn_01x02_Pin(xt60), J6 OLED DISPLAY, J7 EC5 JUMP CONNECTOR, J8 GSB4111312HR, J9 Conn_01x01_Pin, Q1 SIR680LDP-T1-RE3, Q2 SIR680LDP-T1-RE3, Q3 SIR680LDP-T1-RE3, Q4 SIR680LDP-T1-RE3, Q5 Q_PMOS_DGS, Q7 AO3401A, Q8 2N7002, SW1 SW_Push, SW2 SW_Push, U1 BQ25756ERRVR, U2 LMR51420XDDCR, U3 MCP45HV51-ST, U4 INA226, U5 LM317_TO3, U6 TLV76133KVUR, U7 TLV61047DDC

Commit message: 10.30.2026 New Cap footprints
Parts:
- removed C28, C6: 56uF, 80V, Capacitor_THT:CP_Radial_D10.0mm_P2.50mm, symbol Device:C_Polarized_US
- removed C34, C35: 56uF 80V, Capacitor_THT:CP_Radial_D10.0mm_P2.50mm, symbol Device:C_Polarized_US
- removed C4, C5: 56uF 80v, Capacitor_THT:CP_Radial_D10.0mm_P2.50mm, symbol Device:C_Polarized_US
- removed C40: 220uF 35v, Capacitor_THT:CP_Radial_D10.0mm_P2.50mm, symbol Device:C_Polarized_US
- removed C44, C45: 22uF 16V, Capacitor_THT:CP_Radial_D10.0mm_P2.50mm, symbol Device:C_Polarized_US
- added C28, C34, C35, C4, C5, C6: UPJ1K560MPD6, CAP_UPJ_10X15_NCH, symbol Battguard:UPJ1K560MPD6
- added C40: B41858C7227M000, B41858C7227M000:CAPPRD500W60D1000H1350, symbol Battguard:B41858C7227M000
- added C44, C45: ECA1CM220I, ECA1CM220I:CAPPRD250W50D500H1100, symbol Battguard:ECA1CM220I
Connections:
- net +18.5V: now also U3.14 (V+)
- net +5V: now also C44.P, C45.P
- net GND: now also C28.2, C34.2, C35.2, C4.2, C40.2, C44.N, C45.N, C5.2, C6.2
- net VAC: now also C4.1, C5.1
- net Vout: now also C28.1
- net Vsys: now also C6.1
- net Vsystem: now also C34.1, C35.1, C40.1

Commit message: 10.30.2026 fixed capictor routing, 18.5 feed line setup correctly 12v charge circuit done and cleaned up
Connections:
- net +3V3: now also C58.1, C59.1
- net +5V: no longer C58.1, C59.1
Changed lines of the file:
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@@
 	)
 	(symbol
-		(lib_id "power:+5V")
-		(at 307.34 130.81 0)
-		(unit 1)
-		(body_style 1)
-		(exclude_from_sim no)
-		(in_bom yes)
-		(on_board yes)
-		(in_pos_files yes)
-		(dnp no)
-		(fields_autoplaced yes)
-		(property "Reference" "#PWR075"
-			(at 307.34 134.62 0)
-			(hide yes)
-			(show_name no)
-			(do_not_autoplace no)
-			(effects
-				(font
-					(size 1.27 1.27)
-				)
-			)
-		)
-		(property "Value" "+5V"
-			(at 307.34 125.73 0)
-			(show_name no)
-			(do_not_autoplace no)
-			(effects
-				(font
-					(size 1.27 1.27)
-				)
-			)
-		)
-		(property "Footprint" ""
-			(at 307.34 130.81 0)
-			(hide yes)
-			(show_name no)
-			(do_not_autoplace no)
-			(effects
-				(font
-					(size 1.27 1.27)
-				)
-			)
-		)
-		(property "Datasheet" ""
-			(at 307.34 130.81 0)
-			(hide yes)
-			(show_name no)
-			(do_not_autoplace no)
-			(effects
-				(font
-					(size 1.27 1.27)
-				)
-			)
-		)
-		(property "Description" "Power symbol creates a global label with name \"+5V\""
-			(at 307.34 130.81 0)
-			(hide yes)
-			(show_name no)
-			(do_not_autoplace no)
-			(effects
-				(font
-					(size 1.27 1.27)
-				)
-			)
-		)
-		(pin "1"
-		)
-		(instances
-			(project "BattGuard"
-				(path "/236cbdd7-d83d-4a8e-9ca8-a6b8cdb61d8b"
-					(reference "#PWR075")
-					(unit 1)
-				)
-			)
-		)
-	)
-	(symbol
 		(lib_id "Device:C")
 		(at 49.53 219.71 0)
@@
 	)
 	(symbol
-		(lib_id "power:+5V")
-		(at 317.5 130.81 0)
-		(unit 1)
-		(body_style 1)
-		(exclude_from_sim no)
-		(in_bom yes)
-		(on_board yes)
-		(in_pos_files yes)
-		(dnp no)
-		(fields_autoplaced yes)
-		(property "Reference" "#PWR077"
-			(at 317.5 134.62 0)
-			(hide yes)
-			(show_name no)
-			(do_not_autoplace no)
-			(effects
-				(font
-					(size 1.27 1.27)
-				)
-			)
-		)
-		(property "Value" "+5V"
-			(at 317.5 125.73 0)
-			(show_name no)
-			(do_not_autoplace no)
-			(effects
-				(font
-					(size 1.27 1.27)
-				)
-			)
-		)
-		(property "Footprint" ""
-			(at 317.5 130.81 0)
-			(hide yes)
-			(show_name no)
-			(do_not_autoplace no)
-			(effects
-				(font
-					(size 1.27 1.27)
-				)
-			)
-		)
-		(property "Datasheet" ""
-			(at 317.5 130.81 0)
-			(hide yes)
-			(show_name no)
-			(do_not_autoplace no)
-			(effects
-				(font
-					(size 1.27 1.27)
-				)
-			)
-		)
-		(property "Description" "Power symbol creates a global label with name \"+5V\""
-			(at 317.5 130.81 0)
-			(hide yes)
-			(show_name no)
-			(do_not_autoplace no)
-			(effects
-				(font
-					(size 1.27 1.27)
-				)
-			)
-		)
-		(pin "1"
-		)
-		(instances
-			(project "BattGuard"
-				(path "/236cbdd7-d83d-4a8e-9ca8-a6b8cdb61d8b"
-					(reference "#PWR077")
-					(unit 1)
-				)
-			)
-		)
-	)
-	(symbol
 		(lib_id "Device:R_US")
 		(at 302.26 95.25 90)
@@
 	)
 	(symbol
+		(lib_id "power:+3V3")
+		(at 317.5 130.81 0)
+		(unit 1)
+		(body_style 1)
+		(exclude_from_sim no)
+		(in_bom yes)
+		(on_board yes)
+		(in_pos_files yes)
+		(dnp no)
+		(fields_autoplaced yes)
+		(property "Reference" "#PWR075"
+			(at 317.5 134.62 0)
+			(hide yes)
+			(show_name no)
+			(do_not_autoplace no)
+			(effects
+				(font
+					(size 1.27 1.27)
+				)
+			)
+		)
+		(property "Value" "+3V3"
+			(at 317.5 125.73 0)
+			(show_name no)
+			(do_not_autoplace no)
+			(effects
+				(font
+					(size 1.27 1.27)
+				)
+			)
+		)
+		(property "Footprint" ""
+			(at 317.5 130.81 0)
+			(hide yes)
+			(show_name no)
+			(do_not_autoplace no)
+			(effects
+				(font
+					(size 1.27 1.27)
+				)
+			)
+		)
+		(property "Datasheet" ""
+			(at 317.5 130.81 0)
+			(hide yes)
+			(show_name no)
+			(do_not_autoplace no)
+			(effects
+				(font
+					(size 1.27 1.27)
+				)
+			)
+		)
+		(property "Description" "Power symbol creates a global label with name \"+3V3\""
+			(at 317.5 130.81 0)
+			(hide yes)
+			(show_name no)
+			(do_not_autoplace no)
+			(effects
+				(font
+					(size 1.27 1.27)
+				)
+			)
+		)
+		(pin "1"
+		)
+		(instances
+			(project "BattGuard"
+				(path "/236cbdd7-d83d-4a8e-9ca8-a6b8cdb61d8b"
+					(reference "#PWR075")
+					(unit 1)
+				)
+			)
+		)
+	)
+	(symbol
 		(lib_id "power:+5V")
 		(at 229.87 195.58 0)
@@
 	)
 	(symbol
+		(lib_id "power:+3V3")
+		(at 307.34 130.81 0)
+		(unit 1)
+		(body_style 1)
+		(exclude_from_sim no)
+		(in_bom yes)
+		(on_board yes)
+		(in_pos_files yes)
+		(dnp no)
+		(fields_autoplaced yes)
+		(property "Reference" "#PWR060"
+			(at 307.34 134.62 0)
+			(hide yes)
+			(show_name no)
+			(do_not_autoplace no)
+			(effects
+				(font
+					(size 1.27 1.27)
+				)
+			)
+		)
+		(property "Value" "+3V3"
+			(at 307.34 125.73 0)
+			(show_name no)
+			(do_not_autoplace no)
+			(effects
+				(font
+					(size 1.27 1.27)
+				)
+			)
+		)
+		(property "Footprint" ""
+			(at 307.34 130.81 0)
+			(hide yes)
+			(show_name no)
+			(do_not_autoplace no)
+			(effects
+				(font
+					(size 1.27 1.27)
+				)
+			)
+		)
+		(property "Datasheet" ""
+			(at 307.34 130.81 0)
+			(hide yes)
+			(show_name no)
+			(do_not_autoplace no)
+			(effects
+				(font
+					(size 1.27 1.27)
+				)
+			)
+		)
+		(property "Description" "Power symbol creates a global label with name \"+3V3\""
+			(at 307.34 130.81 0)
+			(hide yes)
+			(show_name no)
+			(do_not_autoplace no)
+			(effects
+				(font
+					(size 1.27 1.27)
+				)
+			)
+		)
+		(pin "1"
+		)
+		(instances
+			(project "BattGuard"
+				(path "/236cbdd7-d83d-4a8e-9ca8-a6b8cdb61d8b"
+					(reference "#PWR060")
+					(unit 1)
+				)
+			)
+		)
+	)
+	(symbol
 		(lib_id "Device:R_US")
 		(at 392.43 186.69 0)
@@
 		(exclude_from_sim no)
 		(in_bom yes)
-		(on_board yes)
+		(on_board no)
 		(in_pos_files yes)
 		(dnp no)
