File: board/BattGuard/ESP32-Devboard.kicad_pcb (KiCad board)
At the start: 2 copper layers, 0 parts

Commit message: ESP32 Devboard Update
STEP File and PCB Update
Parts:
- added REF**: ESP32-S3-WROOM-2, RF_Module:ESP32-S3-WROOM-2, F.Cu at (151.0, 84.4)
- added REF**: PinHeader_1x22_P2.54mm_Vertical, Connector_PinHeader_2.54mm:PinHeader_1x22_P2.54mm_Vertical, B.Cu at (162.3, 79.5)
- added REF**: PinHeader_1x22_P2.54mm_Vertical, Connector_PinHeader_2.54mm:PinHeader_1x22_P2.54mm_Vertical, B.Cu at (139.5, 79.6)
